Commit message: 🔧 优化相机位置：将相机移动到船头位置，解决视野遮挡问题
- 将相机位置从 xyz(0.8, 0, 0.05) 调整到 xyz(1.2, 0, 0)
- 调整鼻锥位置从 xyz(1.1, 0, 0) 到 xyz(0.9, 0, 0)，避免遮挡相机
- 调整声纳位置从 xyz(0.6, 0, -0.08) 到 xyz(0.4, 0, -0.08)
- 确保相机视野无遮挡，提高SLAM系统性能
- 更新RViz配置文件，优化分屏布局显示效果

File: src/dolphin_slam/urdf/auv_robot.xacro (robot description, xacro)
@@ -56,5 +56,5 @@
     <parent link="base_link"/>
     <child link="camera_link"/>
-    <origin xyz="0.8 0 0.05" rpy="0 0 0"/>
+    <origin xyz="1.2 0 0" rpy="0 0 0"/>
   </joint>
   <!-- 其他传感器连接 -->
@@ -100,5 +100,5 @@
     <parent link="base_link"/>
     <child link="sonar_link"/>
-    <origin xyz="0.6 0 -0.08" rpy="0 0 0"/>
+    <origin xyz="0.4 0 -0.08" rpy="0 0 0"/>
   </joint>
   <link name="dvl_link">
@@ -248,5 +248,5 @@
     <parent link="base_link"/>
     <child link="nose_cone"/>
-    <origin xyz="1.1 0 0" rpy="0 0 0"/>
+    <origin xyz="0.9 0 0" rpy="0 0 0"/>
   </joint>
   <!-- Gazebo 材质配置 -->
